Commit message: successfully loaded rbd digit

File: src/robots/digit/models/digit_w_grippers.urdf (robot description, URDF)
Before this commit: robot digit, 31 links, 30 joints
Links:
- link left_hip_pitch: geometry collision mesh filename=package://hip-pitch.obj; visual mesh filename=package://hip-pitch.obj
- link left_hip_roll: geometry collision mesh filename=package://hip-yaw-housing.obj; visual mesh filename=package://hip-yaw-housing.obj
- link left_hip_yaw: geometry collision mesh filename=package://hip-pitch-housing.obj; visual mesh filename=package://hip-pitch-housing.obj
- link left_knee: geometry collision mesh filename=package://knee.obj; visual mesh filename=package://knee.obj
- link left_shin: geometry collision mesh filename=package://shin.obj; visual mesh filename=package://shin.obj
- link left_tarsus: geometry collision mesh filename=package://tarsus.obj; visual mesh filename=package://tarsus.obj
- link left_toe_pitch: geometry collision mesh filename=package://toe-pitch.obj; visual mesh filename=package://toe-pitch.obj
- link left_toe_roll: geometry collision mesh filename=package://toe-roll.obj; visual mesh filename=package://toe-roll.obj
- link right_hip_pitch: geometry collision mesh filename=package://hip-pitch.obj scale=1 -1 1; visual mesh filename=package://hip-pitch.obj scale=1 -1 1
- link right_hip_roll: geometry collision mesh filename=package://hip-yaw-housing.obj scale=1 -1 1; visual mesh filename=package://hip-yaw-housing.obj scale=1 -1 1
- link right_hip_yaw: geometry collision mesh filename=package://hip-pitch-housing.obj scale=1 -1 1; visual mesh filename=package://hip-pitch-housing.obj scale=1 -1 1
- link right_knee: geometry collision mesh filename=package://knee.obj scale=1 -1 1; visual mesh filename=package://knee.obj scale=1 -1 1
- link right_shin: geometry collision mesh filename=package://shin.obj scale=1 -1 1; visual mesh filename=package://shin.obj scale=1 -1 1
- link right_tarsus: geometry collision mesh filename=package://tarsus.obj scale=1 -1 1; visual mesh filename=package://tarsus.obj scale=1 -1 1
- link right_toe_pitch: geometry collision mesh filename=package://toe-pitch.obj scale=1 -1 1; visual mesh filename=package://toe-pitch.obj scale=1 -1 1
- link right_toe_roll: geometry collision mesh filename=package://toe-roll.obj scale=1 -1 1; visual mesh filename=package://toe-roll.obj scale=1 -1 1

Commit message: added pads beneath feet

File: src/robots/digit/models/digit_w_grippers.urdf (robot description, URDF)
Before this commit: robot digit, 31 links, 30 joints
Links:
- added link leftpin, mass 0.5; collision box size=0.3 0.1 0.015; visual box size=0.3 0.1 0.015
- added link rightpin, mass 0.5; collision box size=0.3 0.1 0.015; visual box size=0.3 0.1 0.015
Joints:
- added joint leftpinjoint: type fixed, parent left_toe_roll, child leftpin, origin xyz=0.0 -0.065 -0.025 rpy=0 -1.05 -1.57
- added joint rightpinjoint: type fixed, parent right_toe_roll, child rightpin, origin xyz=0.0 0.065 -0.025 rpy=0 -1.05 1.57

Commit message: posture controller working

File: src/robots/digit/models/digit_w_grippers.urdf (robot description, URDF)
Before this commit: robot digit, 33 links, 32 joints
Links:
- link leftpin: geometry collision box size=0.5 0.1 0.015; visual box size=0.5 0.1 0.015
- link rightpin: geometry collision box size=0.5 0.1 0.015; visual box size=0.5 0.1 0.015

Commit message: cleaned up simulator

File: src/robots/digit/models/digit_w_grippers.urdf (robot description, URDF)
Before this commit: robot digit, 33 links, 32 joints
Links:
- link leftpin: geometry collision box size=0.3 0.1 0.015; visual box size=0.3 0.1 0.015
- link rightpin: geometry collision box size=0.3 0.1 0.015; visual box size=0.3 0.1 0.015

File: src/robots/picklerick/model/picklerick.urdf (robot description, URDF)
Before this commit: robot picklerick, 16 links, 15 joints
Joints:
- joint left_elbow_yaw: type continuous -> revolute
- joint left_hip_pitch: type continuous -> revolute
- joint left_shin_yaw: type continuous -> revolute
- joint left_shoulder_pitch: type continuous -> revolute
- joint left_shoulder_yaw: type continuous -> revolute
- joint left_thigh_yaw: type continuous -> revolute
- joint right_elbow_yaw: type continuous -> revolute
- joint right_hip_pitch: type continuous -> revolute
- joint right_shin_yaw: type continuous -> revolute
- joint right_shoulder_pitch: type continuous -> revolute
- joint right_shoulder_yaw: type continuous -> revolute
- joint right_thigh_yaw: type continuous -> revolute
